File: boards/programming-carrier/carrier.kicad_sch (KiCad schematic)
At the start: 149 parts, among them J1 DF40C-40DP-0.4V(51), J2 DF40C(2.0)-40DS-0.4V(51), J3 USB-C USB2, SW1 BOOT / RUN, SW2 RESET, SW3 GPIO46 INPUT, U1 AP2112K-3.3, U10 SN74LVC541APWR, U2 USBLC6-2SC6, U3 SN74LVC541APWR, U4 SN74LVC541APWR, U5 SN74LVC541APWR, U6 SN74LVC541APWR, U7 SN74LVC541APWR, U8 SN74LVC541APWR, U9 SN74LVC541APWR

Commit message: Move carrier JLCPCB CPL corrections onto the parts
Replace boards/programming-carrier/docs/jlcpcb-placement-offsets.json with
hidden F.Fab part fields on the symbols and footprints:
JLCPCB Rotation Offset = -90 on U1-U11, and footprint-local
JLCPCB Position Offset = 0,-2.75 on SW1 (0 deg) and 0,-1.425 on J3
(180 deg). carrier_export.py now reads the fields and maps local offsets
to CPL like pad offsets. The regenerated CPL is byte-identical to
releases/v1/CPL_carrier.csv. ERC/DRC with schematic parity stay at 0, and
Gerbers are unchanged apart from timestamps (not recommitted). The frozen
releases/v1 table copy is untouched.

Co-Authored-By: Claude Opus 5.5 <noreply@anthropic.com>
Parts:
- J3: JLCPCB Position Offset (none) -> 0,-1.425
- SW1: JLCPCB Position Offset (none) -> 0,-2.75
- U1, U10, U2, U3, U4, U5, U6, U7, U8, U9: JLCPCB Rotation Offset (none) -> -90
