File: boards/programming-carrier/rgb.kicad_sch (KiCad schematic)
At the start: 16 parts, among them U11 SN74LVC541APWR

Commit message: Move carrier JLCPCB CPL corrections onto the parts
Replace boards/programming-carrier/docs/jlcpcb-placement-offsets.json with
hidden F.Fab part fields on the symbols and footprints:
JLCPCB Rotation Offset = -90 on U1-U11, and footprint-local
JLCPCB Position Offset = 0,-2.75 on SW1 (0 deg) and 0,-1.425 on J3
(180 deg). carrier_export.py now reads the fields and maps local offsets
to CPL like pad offsets. The regenerated CPL is byte-identical to
releases/v1/CPL_carrier.csv. ERC/DRC with schematic parity stay at 0, and
Gerbers are unchanged apart from timestamps (not recommitted). The frozen
releases/v1 table copy is untouched.

Co-Authored-By: Claude Opus 5.5 <noreply@anthropic.com>
Parts:
- U11: JLCPCB Rotation Offset (none) -> -90
