File: boards/gps-time-calibrator/calibrator.kicad_sch (KiCad schematic)
At the start: 313 parts, among them J1 DF40C-40DP-0.4V(51), J2 DF40C(2.0)-40DS-0.4V(51), J3 USB-C 5V/3A + DATA, J5 GPS ANTENNA, J6 INPUT 5V / 2.5V THRESHOLD, J7 FPGA OUTPUT 5V, Q1 AO3400A, Q10 AO3400A, Q11 AO3400A, Q12 AO3400A, Q13 AO3400A, Q14 AO3400A, Q15 AO3400A, Q16 AO3400A, Q2 AO3400A, Q3 AO3400A, Q4 AO3400A, Q5 AO3400A, Q6 AO3400A, Q7 AO3400A, Q8 AO3400A, Q9 AO3400A, U1 USBLC6-2SC6, U10 SN74AHCT1G125DBVR, U11 TUSB320LAIRWBR, U12 AP2112K-3.3, U13 SN74LVC1G02DCKR, U14 TPS259531DSGR, U15 TPS62160DGKR, U2 AP2112K-3.3, U3 SN74LVC541APWR, U4 SN74LVC541APWR, U5 AP2112K-3.3, U6 MAX-M10S-00B-01, U7 SN74LVC1G17DBVR, U8 TPS2553DBVR, U9 TLV3501AIDBVR, Y1 AOC97FAJC-10.0000

Commit message: Preserve GPS calibrator RFC v1 and fabrication review snapshot
Parts:
- removed C12: 100nF, Calibrator:C_0805_2012Metric, symbol Calibrator:C12
- removed C67: 100nF, Calibrator:C_0805_2012Metric, symbol Calibrator:C67
- removed C72: 22uF / 25V, Calibrator:C_0805_2012Metric, symbol Calibrator:C72
- removed L2: 2.2uH, Calibrator:L4_L_XFL3012_222MEC, symbol Calibrator:L2
- removed R141: 100k, Calibrator:R_0805_2012Metric, symbol Calibrator:R141
- removed R142: 100k, Calibrator:R_0805_2012Metric, symbol Calibrator:R142
- removed R143: 100k, Calibrator:R_0805_2012Metric, symbol Calibrator:R143
- removed R144: 100k, Calibrator:R_0805_2012Metric, symbol Calibrator:R144
- removed R145: 100k, Calibrator:R_0805_2012Metric, symbol Calibrator:R145
- removed R146: 100k, Calibrator:R_0805_2012Metric, symbol Calibrator:R146
- removed R147: 100k, Calibrator:R_0805_2012Metric, symbol Calibrator:R147
- removed R148: 100k, Calibrator:R_0805_2012Metric, symbol Calibrator:R148
- removed R149: 100k, Calibrator:R_0805_2012Metric, symbol Calibrator:R149
- removed R150: 100k, Calibrator:R_0805_2012Metric, symbol Calibrator:R150
- removed R151: 100k, Calibrator:R_0805_2012Metric, symbol Calibrator:R151
- removed R152: 100k, Calibrator:R_0805_2012Metric, symbol Calibrator:R152
- removed R153: 100k, Calibrator:R_0805_2012Metric, symbol Calibrator:R153
- removed R154: 100k, Calibrator:R_0805_2012Metric, symbol Calibrator:R154
- removed R155: 100k, Calibrator:R_0805_2012Metric, symbol Calibrator:R155
- removed R165: 300k, Calibrator:R_0805_2012Metric, symbol Calibrator:R165
- removed R166: 300k, Calibrator:R_0805_2012Metric, symbol Calibrator:R166
- removed R171: 75kR, Calibrator:R_0805_2012Metric, symbol Calibrator:R171
- removed R172: 24kR, Calibrator:R_0805_2012Metric, symbol Calibrator:R172
- removed U13: SN74LVC1G02DCKR, Calibrator:SOT-353_SC-70-5, symbol Calibrator:U13
- removed U8: TPS2553DBVR, Calibrator:SOT-23-6_U8, symbol Calibrator:U8
- added C78: 100nF, Calibrator:C_0805_2012Metric, symbol Calibrator:C78
- added D74: GREEN, Calibrator:LED_0603_1608Metric, symbol Calibrator:D74
- added J8: 61300411121, Calibrator:OLED_Header_1x04_P2.54mm, symbol Calibrator:J8
- added R176: 100k, Calibrator:R_0805_2012Metric, symbol Calibrator:R176
- added R177: 100k, Calibrator:R_0805_2012Metric, symbol Calibrator:R177
- added R178: 100k, Calibrator:R_0805_2012Metric, symbol Calibrator:R178
- added R179: 1k, Calibrator:R_0805_2012Metric, symbol Calibrator:R179
- added R180: 33R, Calibrator:R_0805_2012Metric, symbol Calibrator:R180
- added TP1: VBUS, Calibrator:TP_1p0mm, symbol Calibrator:TP1
- added TP10: PD_SDA, Calibrator:TP_1p0mm, symbol Calibrator:TP10
- added TP11: PD_SCL, Calibrator:TP_1p0mm, symbol Calibrator:TP11
- added TP12: I_MON, Calibrator:TP_1p0mm, symbol Calibrator:TP12
- added TP13: PPS_SRC, Calibrator:TP_1p0mm, symbol Calibrator:TP13
- added TP14: PPS_FPGA, Calibrator:TP_1p0mm, symbol Calibrator:TP14
- added TP15: PPS_ESP, Calibrator:TP_1p0mm, symbol Calibrator:TP15
- added TP16: CLK_FPGA, Calibrator:TP_1p0mm, symbol Calibrator:TP16
- added TP17: TRIG_FILT, Calibrator:TP_1p0mm, symbol Calibrator:TP17
- added TP18: TRIG_2V5, Calibrator:TP_1p0mm, symbol Calibrator:TP18
- added TP19: TRIG_CMP, Calibrator:TP_1p0mm, symbol Calibrator:TP19
- added TP2: 5V_LOAD, Calibrator:TP_1p0mm, symbol Calibrator:TP2
- added TP20: TRIG_3V3, Calibrator:TP_1p0mm, symbol Calibrator:TP20
- added TP23: OUT_FPGA, Calibrator:TP_1p0mm, symbol Calibrator:TP23
- added TP24: OUT_DRV, Calibrator:TP_1p0mm, symbol Calibrator:TP24
- added TP25: GPS_TX, Calibrator:TP_1p0mm, symbol Calibrator:TP25
- added TP26: GPS_RX, Calibrator:TP_1p0mm, symbol Calibrator:TP26
- added TP27: GPS_RST_N, Calibrator:TP_1p0mm, symbol Calibrator:TP27
- added TP28: ANT_PWR, Calibrator:TP_1p0mm, symbol Calibrator:TP28
- added TP29: ANT_BIAS, Calibrator:TP_1p0mm, symbol Calibrator:TP29
- added TP3: 3V3_LOGIC, Calibrator:TP_1p0mm, symbol Calibrator:TP3
- added TP30: LED_OE_N, Calibrator:TP_1p0mm, symbol Calibrator:TP30
- added TP4: 3V3_CC, Calibrator:TP_1p0mm, symbol Calibrator:TP4
- added TP5: 3V3_GPS, Calibrator:TP_1p0mm, symbol Calibrator:TP5
- added TP6: 3V3_OCXO, Calibrator:TP_1p0mm, symbol Calibrator:TP6
- added TP63: OLED_SCL, Calibrator:TP_1p0mm, symbol Calibrator:TP63
- added TP64: OLED_SDA, Calibrator:TP_1p0mm, symbol Calibrator:TP64
- added TP65: BOOT_N, Calibrator:TP_1p0mm, symbol Calibrator:TP65
- added TP7: LOAD_EN, Calibrator:TP_1p0mm, symbol Calibrator:TP7
- added TP8: OCXO_EN, Calibrator:TP_1p0mm, symbol Calibrator:TP8
- added TP9: GPS_EN, Calibrator:TP_1p0mm, symbol Calibrator:TP9
- C64: value 100nF -> 1uF; LCSC C1711 -> C28323; MPN CL21B104KBCNNNC -> CL21B105KBFNNNE
- C75: LCSC C5375915 -> C29925; MPN TCC0805COG102G500BT -> 0805CG102J500NT
- D10, D11, D12, D13, D14, D15, D16, D17, D18, D19, D20, D21, D22, D23, D24, D25, D26, D27, D28, D29, D30, D31, D32, D33, D34, D35, D36, D37, D38, D39, D40, D41, D42, D43, D44, D45, D46, D47, D48, D49, D50, D51, D52, D53, D54, D55, D56, D57, D58, D59, D60, D61, D62, D63, D64, D65, D66, D67, D68, D69, D70, D71, D72, D73: value BLUE -> GREEN; LCSC C28310438 -> C30584801; MPN YLED1206B -> YLED1206G; Manufacturer (none) -> YONGYUTAI; Supplier URL (none) -> https://www.lcsc.com/product-detail/C30584801.html
- R140: value 100k -> 10k; LCSC C96346 -> C17414; MPN RC0805FR-07100KL -> 0805W8F1002T5E
- R164: value 300k -> 22.6k; LCSC C17616 -> C3016901; MPN 0805W8F3003T5E -> SCR0805F22K6; Manufacturer (none) -> VO; Supplier URL (none) -> https://www.lcsc.com/product-detail/C3016901.html
- R6, R7: value 100R -> 33R; LCSC C105577 -> C17634; MPN RC0805FR-07100RL -> 0805W8F330JT5E
- U11: value TUSB320LAIRWBR -> HUSB238_002DD; footprint Calibrator:Texas_X2QFN-12_1.6x1.6mm_P0.4mm -> Calibrator:HUSB238_DFN10_3x3mm; LCSC C132554 -> C7471904; MPN TUSB320LAIRWBR -> HUSB238_002DD
- U15: value TPS62160DGKR -> TPS7A4533DCQR; footprint Calibrator:U3_VSSOP-8_3x3mm_P0.65mm -> Calibrator:SOT-223-6; LCSC C60726 -> C2877942; MPN TPS62160DGKR -> TPS7A4533DCQR
Connections:
- net OCXO_FB is gone; now on net +3V3_OCXO: U15.5 (SENSE)
- net USB_3A_EN is gone; now on net ESP_GPIO4: R169.1, U14.2 (EN)
- net VBUS_DET is gone; now on net CC1: U11.4 (CC1)
- net VBUS_DET_A is gone; now on net GND: R164.2
- net +3V3_CC: now also TP4.1
- net +3V3_GPS: now also C11.1, U7.5 (VCC), TP5.1
- net +3V3_LOGIC: now also R140.1, J8.2 (VCC), TP3.1; no longer C11.1, DS1.2 (VCC), U7.5 (VCC)
- net +3V3_OCXO: now also U15.4 (OUT), TP6.1; no longer U15.6 (VOS)
- net ANT_BIAS: now also TP29.1
- net ANT_PWR: now also U6.14 (VCC_RF), TP28.1
- net CC1: no longer U11.1 (CC1)
- net CC2: now also U11.5 (CC2); no longer U11.2 (CC2)
- net DRIVE0: now also U4.18 (Y0); no longer U4.11 (Y7)
- net DRIVE1: now also U4.17 (Y1); no longer U4.12 (Y6)
- net DRIVE10: now also U3.16 (Y2); no longer U3.13 (Y5)
- net DRIVE11: now also U3.15 (Y3); no longer U3.14 (Y4)
- net DRIVE12: now also U3.14 (Y4); no longer U3.15 (Y3)
- net DRIVE13: now also U3.13 (Y5); no longer U3.16 (Y2)
- net DRIVE14: now also U3.12 (Y6); no longer U3.17 (Y1)
- net DRIVE15: now also U3.11 (Y7); no longer U3.18 (Y0)
- net DRIVE2: now also U4.16 (Y2); no longer U4.13 (Y5)
- net DRIVE3: now also U4.15 (Y3); no longer U4.14 (Y4)
- net DRIVE4: now also U4.14 (Y4); no longer U4.15 (Y3)
- net DRIVE5: now also U4.13 (Y5); no longer U4.16 (Y2)
- net DRIVE6: now also U4.12 (Y6); no longer U4.17 (Y1)
- net DRIVE7: now also U4.11 (Y7); no longer U4.18 (Y0)
- net DRIVE8: now also U3.18 (Y0); no longer U3.11 (Y7)
- net DRIVE9: now also U3.17 (Y1); no longer U3.12 (Y6)
- net ESP_GPIO0_BOOT: now also TP65.1
- net ESP_GPIO1: now also J8.4 (SDA), TP64.1; no longer DS1.4 (SDA)
- net ESP_GPIO2: now also J8.3 (SCL), TP63.1; no longer DS1.3 (SCL)
- net ESP_GPIO38: now also TP15.1
- net ESP_GPIO43_TXD: now also TP26.1
- net ESP_GPIO44_RXD: now also TP25.1
- net FPGA_IOB_13B: now also U3.6 (A4); no longer U3.5 (A3)
- net FPGA_IOB_16A: now also U3.8 (A6); no longer U3.3 (A1)
- net FPGA_IOB_18A: now also U3.9 (A7); no longer R140.1, U3.2 (A0)
- net FPGA_IOB_20A: now also U3.5 (A3); no longer U3.6 (A4)
- net FPGA_IOB_22A: now also U3.7 (A5); no longer U3.4 (A2)
- net FPGA_IOB_23B: now also U3.3 (A1); no longer U3.7 (A5)
- net FPGA_IOB_25B_G3: now also U4.9 (A7); no longer U3.9 (A7)
- net FPGA_IOB_29B: now also U3.2 (A0); no longer U3.8 (A6)
- net FPGA_IOB_3B_G6: now also TP16.1
- net FPGA_IOT_36B: now also U4.8 (A6); no longer U4.2 (A0)
- net FPGA_IOT_38B: now also U4.7 (A5); no longer U4.3 (A1)
- net FPGA_IOT_39A: now also U4.6 (A4); no longer U4.4 (A2)
- net FPGA_IOT_42B: now also U4.4 (A2); no longer U4.6 (A4)
- net FPGA_IOT_43A: now also U4.3 (A1); no longer U4.7 (A5)
- net FPGA_IOT_46B_G0: now also TP14.1
- net FPGA_IOT_48B: now also U4.2 (A0); no longer U4.8 (A6)
- net FPGA_IOT_51A: now also TP23.1
- net GND: now also U11.8 (VSET), U15.3 (GND), U15.6 (TAB), C78.2, D74.1, J8.1 (GND), R177.2, R178.2; no longer DS1.1 (GND), R140.2, U11.10 (GND), U11.3 (PORT_UFP), U15.1 (PGND), U15.4 (AGND), U3.1 (~OE1), U4.1 (~OE1)
- net GPS_PPS: now also R179.1, TP13.1
- net TRIGGER_3V3: now also TP20.1
- net TRIGGER_5V: now also TP19.1
- net TRIGGER_DRV: now also TP24.1
- net TRIGGER_LIMIT: now also TP17.1
- net TRIGGER_VREF: now also TP18.1
- net USB_ILIM: now also R176.1
- net USB_VBUS: now also C2.1, J1.1, J1.2, J1.3, J1.4, U11.1 (VIN), U2.1 (VIN), U2.3 (EN), TP1.1; no longer R164.1, U11.12 (VDD)
- net VIN_5V: now also TP2.1; no longer C2.1, J1.1, J1.2, J1.3, J1.4, U15.3 (EN), U2.1 (VIN), U2.3 (EN), U5.3 (EN)
- net ESP_GPIO3: now reaches J1.15
- net ESP_GPIO3: now also C78.1, R176.2, TP12.1
- net ESP_GPIO4: now reaches J1.16
- net ESP_GPIO4: now also TP7.1
- net ESP_GPIO5: now reaches J1.17
- net ESP_GPIO5: now also U15.1 (EN), R178.1, TP8.1
- net ESP_GPIO6: now reaches J1.18
- net ESP_GPIO6: now also U5.3 (EN), R177.1, TP9.1
- net USB_PD_SDA: now reaches J1.19
- net USB_PD_SDA: now also R167.2, U11.6 (SDA), TP10.1
- net USB_PD_SCL: now reaches J1.20
- net USB_PD_SCL: now also R168.2, U11.7 (SCL), TP11.1
- net ESP_GPIO40: now reaches J1.21
- net ESP_GPIO40: now also R180.1
- net FPGA_IOT_44B: now reaches J2.33
- net FPGA_IOT_44B: now also R140.2, U3.1 (~OE1), U4.1 (~OE1), TP30.1
- net FPGA_IOT_37A: now reaches J2.9
- net FPGA_IOT_37A: now also U3.4 (A2)
- net PD_ISET: now reaches U11.9 (ISET)
- net PD_ISET: now also R164.1
- net GPS_RESET_N: now reaches U6.9 (RESET_N)
- net GPS_RESET_N: now also R180.2, TP27.1
- removed net CC_OUT1: R167.2, U11.7 (OUT1)
- removed net CC_OUT2: R168.2, U11.8 (OUT2)
- net FPGA_IOT_45A_G1: no longer names the net of J2.24
- net FPGA_IOT_45A_G1: no longer U4.9 (A7)
- removed net OCXO_SW: U15.7 (SW)
- new net PPS_LED_A: D74.2, R179.2
- no-connect marks 53 -> 41
Other:
- note added: "10 MHz OCXO / 3.3 V linear supply"
- note added: "2.1 W max warm-up; ~1.1 W LDO loss at 5 V; allow 3 min."
- note added: "5 V ONLY: VSET grounded / ISET 22.6k = 3 A / I2C 0x08"
- note added: "D+/D- charger detection unused; USB data stays with ESP32"
- note added: "DS1 solders onto J8; GND / VCC / SCL / SDA."
- note added: "Diagnostic probe pads / functional names on PCB / bare copper, no assembly parts"
- note added: "ESP32 PPS / GPIO38"
- note added: "ESP_GPIO4 enables loads; 820R sets ~2.48 A. ADC: 0.226 V/A nominal, switched loads only."
- note added: "FPGA PPS / G0"
- note added: "HS96L03W2C03"
- note added: "Manual-fit AOC97FAJC-10.0000. Clock -> J2.32 / FPGA G6."
- note added: "Module and logic boot from raw 5 V. GPIO7/8 read PD status over I2C; firmware budgets current before enabling loads."
- note added: "OE high: blank. Configure data before OE low."
- note added: "OLED"
- note added: "PPS indicator"
- note added: "SOT-223 heat spreader below OCXO; GPIO5 enables."
- note added: "TP1 / VBUS"
- note added: "TP10 / PD_SDA"
- note added: "TP11 / PD_SCL"
- note added: "TP12 / I_MON"
- note added: "TP13 / PPS_SRC"
- note added: "TP14 / PPS_FPGA"
- note added: "TP15 / PPS_ESP"
- note added: "TP16 / CLK_FPGA"
- note added: "TP17 / TRIG_FILT"
- note added: "TP18 / TRIG_2V5"
- note added: "TP19 / TRIG_CMP"
- note added: "TP2 / 5V_LOAD"
- note added: "TP20 / TRIG_3V3"
- note added: "TP23 / OUT_FPGA"
- note added: "TP24 / OUT_DRV"
- note added: "TP25 / GPS_TX"
- note added: "TP26 / GPS_RX"
- note added: "TP27 / GPS_RST_N"
- note added: "TP28 / ANT_PWR"
- note added: "TP29 / ANT_BIAS"
- note added: "TP3 / 3V3_LOGIC"
- note added: "TP30 / LED_OE_N"
- note added: "TP4 / 3V3_CC"
- note added: "TP5 / 3V3_GPS"
- note added: "TP6 / 3V3_OCXO"
- note added: "TP63 / OLED_SCL"
- note added: "TP64 / OLED_SDA"
- note added: "TP65 / BOOT_N"
- note added: "TP7 / LOAD_EN"
- note added: "TP8 / OCXO_EN"
- note added: "TP9 / GPS_EN"
- note added: "Trigger input / 5 V TTL / threshold ~2.5 V"
- note added: "Trigger output / 5 V TTL"
- note added: "USB-C PD / 5 V, 3 A sink and protected power"
- note removed: "10 MHz OCXO / dedicated 3.3 V buck and clock output"
- note removed: "4 x 16 blue LEDs / individual 470R 1% resistors / all four rows show the same bit / 1 LSB = 1/65536 s = 15.258789 us"
- note removed: "Clock -> J2.32 / FPGA G6. Firmware must use 10 MHz."
- note removed: "External triggers / 5 V I-O / input threshold ~2.5 V"
- note removed: "Main rail enabled only for 3 A advertisement. 820R: ~2.48 A limit; 100nF: ~12 ms soft start."
- note removed: "Manual-fit AOC97FAJC-10.0000 / 2.1 W max warmup / allow 3 min."
- note removed: "No high-voltage PD negotiation. Lower-current sources leave the main board off."
- note removed: "PPS supplies absolute epoch; OCXO supplies the local timebase."
- note removed: "Prototype hardware: firmware, absolute latency, brightness uniformity and power/RF behavior require validation."
- note removed: "RF feed is straight; protected 3.3 V bias is for an active GPS antenna."
- note removed: "SSD1315 / 128x64 / I2C 0x3C"
- note removed: "USB-C / 5 V, 3 A source detection and protected power"
- moved on the sheet: C10, C11, C13, C14, C15, C70, C71, C73, C74, C75, C8, C9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
