File: boards/gps-time-calibrator/calibrator.kicad_sch (KiCad schematic)
At the start: 327 parts, among them J1 DF40C-40DP-0.4V(51), J2 DF40C(2.0)-40DS-0.4V(51), J3 USB-C 5V/3A + DATA, J5 GPS ANTENNA, J6 INPUT 5V / 2.5V THRESHOLD, J7 FPGA OUTPUT 5V, J8 61300411121, Q1 AO3400A, Q10 AO3400A, Q11 AO3400A, Q12 AO3400A, Q13 AO3400A, Q14 AO3400A, Q15 AO3400A, Q16 AO3400A, Q2 AO3400A, Q3 AO3400A, Q4 AO3400A, Q5 AO3400A, Q6 AO3400A, Q7 AO3400A, Q8 AO3400A, Q9 AO3400A, U1 USBLC6-2SC6, U10 SN74AHCT1G125DBVR, U11 HUSB238_002DD, U12 AP2112K-3.3, U14 TPS259531DSGR, U15 TPS7A4533DCQR, U2 AP2112K-3.3, U3 SN74LVC541APWR, U4 SN74LVC541APWR, U5 AP2112K-3.3, U6 MAX-M10S-00B-01, U7 SN74LVC1G17DBVR, U9 TLV3501AIDBVR, Y1 AOC97FAJC-10.0000

Commit message: Give every display LED its own 100 nF bypass
Only the top of each column had a 100 nF (C20-C35, above row 1) and the
bottom a 10 uF (C40-C55), so the four LEDs in a column saw different local
supply impedance at turn-on. Each of the 64 LEDs now has an identical
0805 100 nF beside its 470R, VIN via below and GND via above: C20-C35
move down to row 1, and C80-C127 are new for rows 2-4. C40-C55 stay as
per-column 10 uF reservoirs.

circuit.json gains the 48 parts. The schematic generator draws each
branch's cap off its VIN tap (DRIVE labels moved below the gate resistor
to make room) and the PDF is re-exported. Part descriptions and README
are updated.

ERC 0; DRC 0 with 0 parity issues (375 parts). Lint adds only 96
info-level via-role notes, one pair per new cap. The quality tool's
bypass-distance count balloons (every VIN_5V cap is measured against every
VIN_5V pin). Its new silk-over-copper hits pair labels with pads ~20 mm
away; native DRC (silk_over_copper = error) and the render show none.

Co-Authored-By: Claude Opus 5.5 <noreply@anthropic.com>
Parts:
- added C100: 100nF, Calibrator:C_0805_2012Metric, symbol Calibrator:C100
- added C101: 100nF, Calibrator:C_0805_2012Metric, symbol Calibrator:C101
- added C102: 100nF, Calibrator:C_0805_2012Metric, symbol Calibrator:C102
- added C103: 100nF, Calibrator:C_0805_2012Metric, symbol Calibrator:C103
- added C104: 100nF, Calibrator:C_0805_2012Metric, symbol Calibrator:C104
- added C105: 100nF, Calibrator:C_0805_2012Metric, symbol Calibrator:C105
- added C106: 100nF, Calibrator:C_0805_2012Metric, symbol Calibrator:C106
- added C107: 100nF, Calibrator:C_0805_2012Metric, symbol Calibrator:C107
- added C108: 100nF, Calibrator:C_0805_2012Metric, symbol Calibrator:C108
- added C109: 100nF, Calibrator:C_0805_2012Metric, symbol Calibrator:C109
- added C110: 100nF, Calibrator:C_0805_2012Metric, symbol Calibrator:C110
- added C111: 100nF, Calibrator:C_0805_2012Metric, symbol Calibrator:C111
- added C112: 100nF, Calibrator:C_0805_2012Metric, symbol Calibrator:C112
- added C113: 100nF, Calibrator:C_0805_2012Metric, symbol Calibrator:C113
- added C114: 100nF, Calibrator:C_0805_2012Metric, symbol Calibrator:C114
- added C115: 100nF, Calibrator:C_0805_2012Metric, symbol Calibrator:C115
- added C116: 100nF, Calibrator:C_0805_2012Metric, symbol Calibrator:C116
- added C117: 100nF, Calibrator:C_0805_2012Metric, symbol Calibrator:C117
- added C118: 100nF, Calibrator:C_0805_2012Metric, symbol Calibrator:C118
- added C119: 100nF, Calibrator:C_0805_2012Metric, symbol Calibrator:C119
- added C120: 100nF, Calibrator:C_0805_2012Metric, symbol Calibrator:C120
- added C121: 100nF, Calibrator:C_0805_2012Metric, symbol Calibrator:C121
- added C122: 100nF, Calibrator:C_0805_2012Metric, symbol Calibrator:C122
- added C123: 100nF, Calibrator:C_0805_2012Metric, symbol Calibrator:C123
- added C124: 100nF, Calibrator:C_0805_2012Metric, symbol Calibrator:C124
- added C125: 100nF, Calibrator:C_0805_2012Metric, symbol Calibrator:C125
- added C126: 100nF, Calibrator:C_0805_2012Metric, symbol Calibrator:C126
- added C127: 100nF, Calibrator:C_0805_2012Metric, symbol Calibrator:C127
- added C80: 100nF, Calibrator:C_0805_2012Metric, symbol Calibrator:C80
- added C81: 100nF, Calibrator:C_0805_2012Metric, symbol Calibrator:C81
- added C82: 100nF, Calibrator:C_0805_2012Metric, symbol Calibrator:C82
- added C83: 100nF, Calibrator:C_0805_2012Metric, symbol Calibrator:C83
- added C84: 100nF, Calibrator:C_0805_2012Metric, symbol Calibrator:C84
- added C85: 100nF, Calibrator:C_0805_2012Metric, symbol Calibrator:C85
- added C86: 100nF, Calibrator:C_0805_2012Metric, symbol Calibrator:C86
- added C87: 100nF, Calibrator:C_0805_2012Metric, symbol Calibrator:C87
- added C88: 100nF, Calibrator:C_0805_2012Metric, symbol Calibrator:C88
- added C89: 100nF, Calibrator:C_0805_2012Metric, symbol Calibrator:C89
- added C90: 100nF, Calibrator:C_0805_2012Metric, symbol Calibrator:C90
- added C91: 100nF, Calibrator:C_0805_2012Metric, symbol Calibrator:C91
- added C92: 100nF, Calibrator:C_0805_2012Metric, symbol Calibrator:C92
- added C93: 100nF, Calibrator:C_0805_2012Metric, symbol Calibrator:C93
- added C94: 100nF, Calibrator:C_0805_2012Metric, symbol Calibrator:C94
- added C95: 100nF, Calibrator:C_0805_2012Metric, symbol Calibrator:C95
- added C96: 100nF, Calibrator:C_0805_2012Metric, symbol Calibrator:C96
- added C97: 100nF, Calibrator:C_0805_2012Metric, symbol Calibrator:C97
- added C98: 100nF, Calibrator:C_0805_2012Metric, symbol Calibrator:C98
- added C99: 100nF, Calibrator:C_0805_2012Metric, symbol Calibrator:C99
Connections:
- net GND: now also C100.2, C101.2, C102.2, C103.2, C104.2, C105.2, C106.2, C107.2, C108.2, C109.2, C110.2, C111.2, C112.2, C113.2, C114.2, C115.2, C116.2, C117.2, C118.2, C119.2, C120.2, C121.2, C122.2, C123.2, C124.2, C125.2, C126.2, C127.2, C80.2, C81.2, C82.2, C83.2, C84.2, C85.2, C86.2, C87.2, C88.2, C89.2, C90.2, C91.2, C92.2, C93.2, C94.2, C95.2, C96.2, C97.2, C98.2, C99.2
- net VIN_5V: now also C100.1, C101.1, C102.1, C103.1, C104.1, C105.1, C106.1, C107.1, C108.1, C109.1, C110.1, C111.1, C112.1, C113.1, C114.1, C115.1, C116.1, C117.1, C118.1, C119.1, C120.1, C121.1, C122.1, C123.1, C124.1, C125.1, C126.1, C127.1, C80.1, C81.1, C82.1, C83.1, C84.1, C85.1, C86.1, C87.1, C88.1, C89.1, C90.1, C91.1, C92.1, C93.1, C94.1, C95.1, C96.1, C97.1, C98.1, C99.1
Other:
- moved on the sheet: C20, C21, C22, C23, C24, C25, C26, C27, C28, C29, C30, C31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

Commit message: Stack the trigger input RC horizontally and drop TP17
C75 (1 nF) and R9 (100k) now lie horizontal directly above R8 at 2.0 mm
pitch, left pads aligned on one short TRIGGER_LIMIT bus to U9 pin 3, GND
pads on the right into the pour. TP17 (TRIG_FILT) is removed from the
board, circuit.json, the regenerated schematic, the testpoint map/CSV/
JSON/audit, final placements and the integration notes. Pad count is now
30 (README said 33, testpoints.md 31).

ERC 0, DRC 0 with 0 parity issues (374 parts); lint 677 -> 671 (six
TRIGGER_LIMIT findings gone, none added); quality warnings 14338 -> 14335.

Co-Authored-By: Claude Opus 5.5 <noreply@anthropic.com>
Parts:
- removed TP17: TRIG_FILT, Calibrator:TP_1p0mm, symbol Calibrator:TP17
Other:
- note removed: "TP17 / TRIG_FILT"

Commit message: Line up the GPS passives beside U6, stand R5 above C10, drop TP28/TP29
R177, R7, R6, C9 and C8 now share one column at x 175.2 mm. The resistors
moved right onto the decoupling caps' line so C9/C8 stay tight to U6. The
GPS_PPS In1 via that would have sat in R6.1 moves to the gap between R7 and
R6, and the +3V3_GPS B.Cu feed via moves onto the C9 -> U6.6 trace.

R5 (antenna bias, 1206) is vertical in the C10/L1 column: ANT_BIAS drops
straight from R5.2 through C10 to L1, and ANT_PWR leaves U6.14 square and
climbs at x 189.6 into R5.1. TP28 (ANT_PWR) and TP29 (ANT_BIAS) are removed
from the board, circuit.json, the regenerated schematic/PDF, the testpoint
map/CSV/JSON/audit, final placements and part descriptions; 28 pads remain.

ERC 0, DRC 0 with 0 parity issues; lint 668 -> 665 (none added); quality
warnings 14335 -> 14331, errors unchanged at 64.

Co-Authored-By: Claude Opus 5.5 <noreply@anthropic.com>
Parts:
- removed TP28: ANT_PWR, Calibrator:TP_1p0mm, symbol Calibrator:TP28
- removed TP29: ANT_BIAS, Calibrator:TP_1p0mm, symbol Calibrator:TP29
Other:
- note removed: "TP28 / ANT_PWR"
- note removed: "TP29 / ANT_BIAS"

Commit message: Drop the 3V3_CC LDO and pull the PD I2C lines up to 3V3_LOGIC
U12 existed only to power R167/R168, the 10k pull-ups on the HUSB238
SDA/SCL. +3V3_LOGIC (U2) is equally always-on from VBUS and is the ESP's own
I/O rail, so the pull-ups now go there and U12, C65, C66 and TP4 are removed.
On the board the pull-up rail runs west on F.Cu into the existing 3V3_LOGIC
via that feeds R4; the U12 pin loop and its three vias are gone.

Schematic, symbol library and PDF regenerated; circuit.json, placements,
part descriptions, power-domain diagram, power/HUSB238/integration notes and
the testpoint map/CSV/JSON/audit updated (27 pads).

ERC 0, DRC 0 / 0 unconnected / 0 parity; lint 631 -> 627; quality errors
68 -> 67, warnings 14316 -> 14310.

Co-Authored-By: Claude Opus 5.5 <noreply@anthropic.com>
Parts:
- removed C65: 4.7uF, Calibrator:C_0805_2012Metric, symbol Calibrator:C65
- removed C66: 4.7uF, Calibrator:C_0805_2012Metric, symbol Calibrator:C66
- removed TP4: 3V3_CC, Calibrator:TP_1p0mm, symbol Calibrator:TP4
- removed U12: AP2112K-3.3, Calibrator:SOT-23-5_U12, symbol Calibrator:U12
Connections:
- net +3V3_CC is gone; now on net +3V3_LOGIC: R167.1, R168.1
- no-connect marks 41 -> 40
Other:
- note removed: "TP4 / 3V3_CC"

Commit message: Escape CC1/CC2 under the USB-C receptacle on F.Cu
Both CC lines leave J3 eastward beneath the receptacle body, run north
between the shell legs and come round to U11 on the top layer, replacing
the four vias and In1 runs. The nested lanes land swapped at U11 (J3 A5 ->
pin 5, B5 -> pin 4) so they never cross; the HUSB238 resolves orientation
from either CC pin. The A12 shell-ground stub now lands in S1, and S1 gets a
short tie to a stitching via since the lanes cut off its old pour path.

Co-Authored-By: Claude Opus 5.5 <noreply@anthropic.com>
Connections:
- net CC1: now also U11.5 (CC2); no longer U11.4 (CC1)
- net CC2: now also U11.4 (CC1); no longer U11.5 (CC2)

Commit message: Place the BOOT pull-up R4 at J1 and drop the GPIO0 test pad TP65
R4 now stands vertically just north of J1 pin 12: BOOT exits the
connector straight into R4 pad 1 and pad 2 tees into the +3V3_LOGIC
F.Cu strip at y 12.5. The 10 mm BOOT run across the module footprint
and the TP65 probe pad are gone; GPIO0 recovery uses R4 pad 1.

TP65 is removed from circuit.json, the schematic/PDF, part descriptions
and the test-point docs and audit (27 -> 26 pads).

Co-Authored-By: Claude Opus 5.5 <noreply@anthropic.com>
Parts:
- removed TP65: BOOT_N, Calibrator:TP_1p0mm, symbol Calibrator:TP65
Other:
- note removed: "TP65 / BOOT_N"

Commit message: Drop the OLED I2C test points TP63/TP64
SCL and SDA are probed at the J8 header instead. The pads, their F.Cu
links and the two vias they hung off are gone; the SCL B.Cu lane is one
straight segment again. TP63/TP64 are removed from circuit.json, the
regenerated schematic and symbol library, the testpoint map/CSV/JSON/
audit (now 24 pads), final placements, part descriptions and README.

Co-Authored-By: Claude Opus 5.5 <noreply@anthropic.com>
Parts:
- removed TP63: OLED_SCL, Calibrator:TP_1p0mm, symbol Calibrator:TP63
- removed TP64: OLED_SDA, Calibrator:TP_1p0mm, symbol Calibrator:TP64
Other:
- note removed: "TP63 / OLED_SCL"
- note removed: "TP64 / OLED_SDA"
