File: boards/tesla-coil-controller/controller.kicad_pcb (KiCad board)
At the start: 2 copper layers, 163 x 141.8 mm, 331 parts, among them J1 DF40C-40DP-0.4V(51), J10 AUX 4 / 0-5V, J2 DF40C(2.0)-40DS-0.4V(51), J3 AUX 1 / 0-5V, J30 12V BATTERY / LOWER, J4 12V BATTERY / UPPER, J40 CST SECONDARY, J5 USB-C / PROGRAMMING ONLY, J50 GDT 1 PRIMARY, J51 GDT 2 PRIMARY, J60 CST 2 SECONDARY, J8 AUX 2 / 0-5V, J9 AUX 3 / 0-5V, Q50 STD80N10F7, Q51 STD80N10F7, Q52 STD80N10F7, Q53 STD80N10F7, Q54 STD80N10F7, Q55 STD80N10F7, Q56 STD80N10F7, Q57 STD80N10F7, U1 AD7606C-16BSTZ, U2 AP2112K-3.3, U3 USBLC6-2SC6, U30 LMZ14202HTZX/NOPB, U31 LMZ14202HTZX/NOPB, U40 OPA197IDBVR, U41 OPA197IDBVR, U42 TLV3501AIDBVR, U44 TPS60403DBVR, U51 UCC27282DR, U52 UCC27282DR, U53 UCC27282DR, U54 UCC27282DR, U60 OPA197IDBVR, U61 OPA197IDBVR, U62 TLV3501AIDBVR, U70 OPA197IDBVR, U71 OPA197IDBVR, U72 OPA197IDBVR, U73 OPA197IDBVR

Commit message: Fold the AUX3 shunt parts horizontal above and below R720
Portal edit-stack item: "Fold the up/down resistors here to be above/below
the left-right one". On the AUX3 input filter the two vertical shunt
parts at x=34 (C720 150 pF above the line, R721 1 MOhm below it) now lie
horizontal in a column with the 1 kOhm series resistor R720: C720 at
(37.14,97.85) and R721 at (37.1,102.15), both pad 1 on the left so the
three signal pads sit on one x=36.19 vertical through R720 pad 1. The
old stub from the line down to the shunt pair is replaced by that one
column segment. Each ground pad now runs straight to its own via: C720
up to (38.09,96.75), R721 down to (38.01,103.56). C721's ground stub,
which used to run left into the space C720 now occupies, goes up to a
via at (40,96.75) instead, mirroring C720.

Generator-owned: tesla_placement.json and tesla_reviewed_routing.json
edited and replayed. Only C720 and R721 moved; only AUX3_0_5V and GND
copper changed. DRC 0/0/0 (kicad-cli and kicadmium). kct lint: 0 open,
no new findings; evidence refreshed for all 178 exceptions.

Co-Authored-By: Claude Fable 5.1 <noreply@anthropic.com>
Parts:
- moved C720 3.36 mm to (37.1, 97.8), turned to 0 degrees
- moved R721 3.14 mm to (37.1, 102.2), turned to 0 degrees
Routing:
- net AUX3_0_5V: track 11.6 -> 14.2 mm
- net GND: track 364.9 -> 364.2 mm
Changed lines of the file:
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@@
 	(footprint "Tesla:C_0805_2012Metric"
 		(layer "F.Cu")
-		(at 34 99.05 90)
+		(at 37.1375 97.85)
 		(descr "Capacitor SMD 0805 (2012 Metric), square (rectangular) end terminal, IPC_7351 nominal, (Body size source: IPC-SM-782 page 76, https://www.pcb-3d.com/wordpress/wp-content/uploads/ipc-sm-782a_amendment_1_and_2.pdf, https://docs.google.com/spreadsheets/d/1BsfQQcO9C6DZCsRaXUlFlo91Tg2WpOkGARC1WS5S8t0/edit?usp=sharing), generated with kicad-footprint-generator")
 		(tags "capacitor")
 		(property "Reference" "C720"
-			(at 0 0 0)
+			(at 0 0 270)
 			(layer "F.SilkS")
 			(hide yes)
@@
 		)
 		(property "Value" "150pF 50V C0G"
-			(at 0 1.68 90)
+			(at 0 1.68 0)
 			(layer "F.Fab")
 			(hide yes)
@@
 		)
 		(property "Datasheet" ""
-			(at 0 0 90)
+			(at 0 0 0)
 			(layer "F.Fab")
 			(hide yes)
@@
 		)
 		(property "Description" ""
-			(at 0 0 90)
+			(at 0 0 0)
 			(layer "F.Fab")
 			(hide yes)
@@
 		)
 		(property "MPN" ""
-			(at 0 0 90)
+			(at 0 0 0)
 			(layer "F.SilkS")
 			(hide yes)
@@
 		)
 		(property "LCSC" ""
-			(at 0 0 90)
+			(at 0 0 0)
 			(layer "F.SilkS")
 			(hide yes)
@@
 		)
 		(property "Design status" "Acquisition draft / not for fabrication"
-			(at 0 0 90)
+			(at 0 0 0)
 			(layer "F.SilkS")
 			(hide yes)
@@
 		)
 		(fp_line
-			(start 1.7 -0.98)
-			(end 1.7 0.98)
+			(start -1.7 -0.98)
+			(end 1.7 -0.98)
 			(stroke
 				(width 0.05)
@@
 		)
 		(fp_line
-			(start -1.7 -0.98)
-			(end 1.7 -0.98)
+			(start -1.7 0.98)
+			(end -1.7 -0.98)
 			(stroke
 				(width 0.05)
@@
 		)
 		(fp_line
-			(start 1.7 0.98)
-			(end -1.7 0.98)
+			(start 1.7 -0.98)
+			(end 1.7 0.98)
 			(stroke
 				(width 0.05)
@@
 		)
 		(fp_line
-			(start -1.7 0.98)
-			(end -1.7 -0.98)
+			(start 1.7 0.98)
+			(end -1.7 0.98)
 			(stroke
 				(width 0.05)
@@
 		)
 		(fp_line
-			(start 1 -0.625)
-			(end 1 0.625)
+			(start -1 -0.625)
+			(end 1 -0.625)
 			(stroke
 				(width 0.1)
@@
 		)
 		(fp_line
-			(start -1 -0.625)
-			(end 1 -0.625)
+			(start -1 0.625)
+			(end -1 -0.625)
 			(stroke
 				(width 0.1)
@@
 		)
 		(fp_line
-			(start 1 0.625)
-			(end -1 0.625)
+			(start 1 -0.625)
+			(end 1 0.625)
 			(stroke
 				(width 0.1)
@@
 		)
 		(fp_line
-			(start -1 0.625)
-			(end -1 -0.625)
+			(start 1 0.625)
+			(end -1 0.625)
 			(stroke
 				(width 0.1)
@@
 		)
 		(fp_text user "${REFERENCE}"
-			(at 0 0 90)
+			(at 0 0 0)
 			(layer "F.Fab")
 			(effects
@@
 		)
 		(pad "1" smd roundrect
-			(at -0.95 0 90)
+			(at -0.95 0)
 			(size 1 1.45)
 			(layers "F.Cu" "F.Mask" "F.Paste")
@@
 		)
 		(pad "2" smd roundrect
-			(at 0.95 0 90)
+			(at 0.95 0)
 			(size 1 1.45)
 			(layers "F.Cu" "F.Mask" "F.Paste")
@@
 	(footprint "Tesla:R_0805_2012Metric"
 		(layer "F.Cu")
-		(at 34 102.65 -90)
+		(at 37.1 102.15)
 		(descr "Resistor SMD 0805 (2012 Metric), square (rectangular) end terminal, IPC_7351 nominal, (Body size source: IPC-SM-782 page 72, https://www.pcb-3d.com/wordpress/wp-content/uploads/ipc-sm-782a_amendment_1_and_2.pdf), generated with kicad-footprint-generator")
 		(tags "resistor")
 		(property "Reference" "R721"
-			(at 0 0 180)
+			(at 0 0 270)
 			(layer "F.SilkS")
 			(hide yes)
@@
 		)
 		(property "Value" "1M 1%"
-			(at 0 1.65 270)
+			(at 0 1.65 0)
 			(layer "F.Fab")
 			(hide yes)
@@
 		)
 		(property "Datasheet" ""
-			(at 0 0 270)
+			(at 0 0 0)
 			(layer "F.Fab")
 			(hide yes)
@@
 		)
 		(property "Description" ""
-			(at 0 0 270)
+			(at 0 0 0)
 			(layer "F.Fab")
 			(hide yes)
@@
 		)
 		(property "MPN" ""
-			(at 0 0 270)
+			(at 0 0 0)
 			(layer "F.SilkS")
 			(hide yes)
@@
 		)
 		(property "LCSC" ""
-			(at 0 0 270)
+			(at 0 0 0)
 			(layer "F.SilkS")
 			(hide yes)
@@
 		)
 		(property "Design status" "Acquisition draft / not for fabrication"
-			(at 0 0 270)
+			(at 0 0 0)
 			(layer "F.SilkS")
 			(hide yes)
@@
 		(duplicate_pad_numbers_are_jumpers no)
 		(fp_line
-			(start -0.227064 0.735)
-			(end 0.227064 0.735)
+			(start -0.227064 -0.735)
+			(end 0.227064 -0.735)
 			(stroke
 				(width 0.12)
@@
 		)
 		(fp_line
-			(start -0.227064 -0.735)
-			(end 0.227064 -0.735)
+			(start -0.227064 0.735)
+			(end 0.227064 0.735)
 			(stroke
 				(width 0.12)
@@
 		)
 		(fp_line
-			(start -1.68 0.95)
-			(end -1.68 -0.95)
+			(start -1.68 -0.95)
+			(end 1.68 -0.95)
 			(stroke
 				(width 0.05)
@@
 		)
 		(fp_line
-			(start 1.68 0.95)
-			(end -1.68 0.95)
+			(start -1.68 0.95)
+			(end -1.68 -0.95)
 			(stroke
 				(width 0.05)
@@
 		)
 		(fp_line
-			(start -1.68 -0.95)
-			(end 1.68 -0.95)
+			(start 1.68 -0.95)
+			(end 1.68 0.95)
 			(stroke
 				(width 0.05)
@@
 		)
 		(fp_line
-			(start 1.68 -0.95)
-			(end 1.68 0.95)
+			(start 1.68 0.95)
+			(end -1.68 0.95)
 			(stroke
 				(width 0.05)
@@
 		)
 		(fp_line
-			(start -1 0.625)
-			(end -1 -0.625)
+			(start -1 -0.625)
+			(end 1 -0.625)
 			(stroke
 				(width 0.1)
@@
 		)
 		(fp_line
-			(start 1 0.625)
-			(end -1 0.625)
+			(start -1 0.625)
+			(end -1 -0.625)
 			(stroke
 				(width 0.1)
@@
 		)
 		(fp_line
-			(start -1 -0.625)
-			(end 1 -0.625)
+			(start 1 -0.625)
+			(end 1 0.625)
 			(stroke
 				(width 0.1)
@@
 		)
 		(fp_line
-			(start 1 -0.625)
-			(end 1 0.625)
+			(start 1 0.625)
+			(end -1 0.625)
 			(stroke
 				(width 0.1)
@@
 		)
 		(fp_text user "${REFERENCE}"
-			(at 0 0 270)
+			(at 0 0 0)
 			(layer "F.Fab")
 			(effects
@@
 		)
 		(pad "1" smd roundrect
-			(at -0.9125 0 270)
+			(at -0.9125 0)
 			(size 1.025 1.4)
 			(layers "F.Cu" "F.Mask" "F.Paste")
@@
 		)
 		(pad "2" smd roundrect
-			(at 0.9125 0 270)
+			(at 0.9125 0)
 			(size 1.025 1.4)
 			(layers "F.Cu" "F.Mask" "F.Paste")
@@
 	)
 	(segment
-		(start 34 103.5625)
-		(end 35.25 103.5625)
+		(start 38.0125 102.15)
+		(end 38.0125 103.5625)
 		(width 0.3)
 		(layer "F.Cu")
@@
 	)
 	(segment
-		(start 34 98.1)
-		(end 34 96.75)
+		(start 38.0875 97.85)
+		(end 38.0875 96.75)
 		(width 0.3)
 		(layer "F.Cu")
@@
 	(segment
 		(start 40 98.1)
-		(end 38.1 98.1)
+		(end 40 96.75)
 		(width 0.3)
 		(layer "F.Cu")
@@
 	)
 	(via
-		(at 34 96.75)
+		(at 38.0875 96.75)
 		(size 0.6)
 		(drill 0.3)
@@
 	)
 	(via
-		(at 35.25 103.5625)
+		(at 38.0125 103.5625)
 		(size 0.6)
 		(drill 0.3)
@@
 	)
 	(via
-		(at 38.1 98.1)
+		(at 40 96.75)
 		(size 0.6)
 		(drill 0.3)
@@
 	)
 	(segment
-		(start 34 100)
-		(end 34 101.7375)
+		(start 36.1875 97.85)
+		(end 36.1875 102.15)
 		(width 0.25)
 		(layer "F.Cu")

Commit message: Run the VBAT bus straight under J1 instead of over the USB area
Portal edit-stack item: "The 12v line takes a too long route here, it can
go below the mcu connector and unsquish the USB". The 2.5 mm VBAT_24V bus
left the y=46 run at x=71.5, climbed to y=37, crossed the whole board
between the USB receptacle J5 and the module connector J1, and came back
down at x=174.85 to the cap bank. The USB D+/D-, VBUS and CC traces had
to thread between that bus and J5.

The y=46 bus now continues straight to x=95, steps down 0.5 mm so it
clears J1's bottom pad row with room for the ground fill, runs at y=46.5
to x=170.85 and takes one 45° to the existing x=174.85 drop, which now
starts above D50's pad and enters it straight. The y=37 run and its two
corners are gone; the diagonal and vertical at x=77 stay as C333's feed.
J1 pad 22 (GND) lost its fill connection under the bus, so its existing
0.2 mm stub now ends in a stitching via at (106.4,44.65). Net bus length
drops by about 11 mm.

Generator-owned: tesla_reviewed_routing.json edited and replayed. No
footprints moved; only VBAT_24V and one GND stub/via changed. DRC 0/0/0
(kicad-cli and kicadmium). kct lint: 0 open. The width-step findings at
the old (71.5,46) corner are resolved because the bus now runs through
that point as a tee; the pre-existing VBAT backtrack at (141,56.35)
re-keyed and is flagged again with its original reason. Evidence
refreshed for the remaining exceptions (121 ignored, 53 flagged).

Co-Authored-By: Claude Fable 5.1 <noreply@anthropic.com>
Routing:
- net VBAT_24V: track 609.7 -> 606.4 mm
- net GND: track 364.2 -> 364.6 mm, vias 198 -> 199
Changed lines of the file:
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@@
 	(segment
 		(start 106.4 44.1)
-		(end 106.4 44.3)
+		(end 106.4 44.65)
 		(width 0.2)
 		(layer "F.Cu")
@@
 	)
 	(via
+		(at 106.4 44.65)
+		(size 0.6)
+		(drill 0.3)
+		(layers "F.Cu" "B.Cu")
+		(net "GND")
+	)
+	(via
 		(at 45.55 30)
 		(size 0.6)
@@
 	(segment
 		(start 36 46)
-		(end 71.525 46)
+		(end 95 46)
 		(width 2.5)
 		(layer "F.Cu")
@@
 	)
 	(segment
-		(start 170 37)
-		(end 174.85 41.85)
+		(start 170.85 46.5)
+		(end 174.85 50.5)
+		(width 2.5)
+		(layer "F.Cu")
+		(net "VBAT_24V")
+	)
+	(segment
+		(start 95 46)
+		(end 95.5 46.5)
+		(width 2.5)
+		(layer "F.Cu")
+		(net "VBAT_24V")
+	)
+	(segment
+		(start 95.5 46.5)
+		(end 170.85 46.5)
 		(width 2.5)
 		(layer "F.Cu")
@@
 	)
 	(segment
-		(start 77.05 37)
-		(end 170 37)
-		(width 2.5)
-		(layer "F.Cu")
-		(net "VBAT_24V")
-	)
-	(segment
 		(start 159 111.35)
 		(end 159 112)
@@
 	)
 	(segment
-		(start 174.85 41.85)
+		(start 174.85 50.5)
 		(end 174.85 57)
 		(width 2.5)

Commit message: Fold the AUX1, AUX2 and AUX4 shunt parts the same way as AUX3
Follow-up to 3bb7e62 at the user's request: the other three AUX input
filters get the identical fold. For each channel (line y = 82, 91, 109)
the vertical shunt cap and shunt resistor at x=34 lie down horizontal in a
column with the series resistor, every signal pad on the x=36.19
vertical through the series resistor's pad 1, and every ground pad going
straight to its own via (cap up, resistor down). The second cap's ground
stub, which used to run left into the space the shunt cap now occupies,
goes up to its own via instead. All four channels are now the same.

Generator-owned: tesla_placement.json and tesla_reviewed_routing.json
edited and replayed. Only C700/R701, C710/R711, C730/R731 moved; only the
AUX*_0_5V and GND copper of those channels changed. DRC 0/0/0 (kicad-cli
and kicadmium). kct lint: 0 open, no new findings; evidence refreshed for
all 174 exceptions.

Co-Authored-By: Claude Fable 5.1 <noreply@anthropic.com>
Parts:
- moved C700 3.36 mm to (37.1, 79.8), turned to 0 degrees
- moved C710 3.36 mm to (37.1, 88.8), turned to 0 degrees
- moved C730 3.36 mm to (37.1, 106.8), turned to 0 degrees
- moved R701 3.14 mm to (37.1, 84.2), turned to 0 degrees
- moved R711 3.14 mm to (37.1, 93.2), turned to 0 degrees
- moved R731 3.14 mm to (37.1, 111.2), turned to 0 degrees
Routing:
- net AUX4_0_5V: track 11.6 -> 14.2 mm
- net AUX2_0_5V: track 11.6 -> 14.2 mm
- net AUX1_0_5V: track 11.6 -> 14.2 mm
- net GND: track 364.6 -> 362.7 mm

Commit message: Fold the CT phase-comparator pull-up, pull-down and cap into R610/R410 columns
User request: "Same transform around R610 and its accomplice" and "C610
could also fold into the line nicely". R610 (CT2) and R410 (CT1) are 17 mm
twins, so both stages get the fold. The vertical pull-up (R611/R411) and
pull-down (R622/R422) at x=97 lie down horizontal above and below the
series resistor at x=94, with every CTn_PHASE pad on the x=94.91 vertical
through the series resistor's pad 2, and the 22 pF cap (C610/C410) joins
the bottom of the same column instead of sitting under the BAT54S with a
diagonal lead. The +3V3 feed line extends left to the pull-up's pad and
drops into it straight; the pull-down and cap grounds each get their own
via. The old x=97 vertical, the diagonal to the cap and the cap's old
ground via are gone.

Generator-owned: tesla_placement.json and tesla_reviewed_routing.json
edited and replayed. Only those six parts moved; only CT1/CT2_PHASE,
+3V3 and GND copper changed. DRC 0/0/0 (kicad-cli and kicadmium). kct
lint: 0 open. Seven findings on the old geometry are resolved (two oblique
pad exits, the D43/D63 detour/backtrack/bend_count flags). Two new +3V3
chain findings on the CT1 feed are flagged with the same backlog reason.

Co-Authored-By: Claude Fable 5.1 <noreply@anthropic.com>
Parts:
- moved C410 6.08 mm to (94.0, 136.3), turned to 180 degrees
- moved C610 6.08 mm to (94.0, 153.3), turned to 180 degrees
- moved R411 3.12 mm to (94.0, 129.8), turned to 0 degrees
- moved R422 3.12 mm to (94.0, 134.2), turned to 180 degrees
- moved R611 3.12 mm to (94.0, 146.8), turned to 0 degrees
- moved R622 3.12 mm to (94.0, 151.2), turned to 180 degrees
Routing:
- net +3V3: track 177.0 -> 185.3 mm
- net CT2_PHASE: track 21.7 -> 20.2 mm
- net CT1_PHASE: track 21.7 -> 20.2 mm
- net GND: track 362.7 -> 361.6 mm
