File: boards/tesla-coil-controller/controller.kicad_sch (KiCad schematic)
At the start: 331 parts, among them J1 DF40C-40DP-0.4V(51), J10 AUX 4 / 0-5V, J2 DF40C(2.0)-40DS-0.4V(51), J3 AUX 1 / 0-5V, J30 12V BATTERY / LOWER, J4 12V BATTERY / UPPER, J40 CST SECONDARY, J5 USB-C / PROGRAMMING ONLY, J50 GDT 1 PRIMARY, J51 GDT 2 PRIMARY, J60 CST 2 SECONDARY, J8 AUX 2 / 0-5V, J9 AUX 3 / 0-5V, Q50 STD80N10F7, Q51 STD80N10F7, Q52 STD80N10F7, Q53 STD80N10F7, Q54 STD80N10F7, Q55 STD80N10F7, Q56 STD80N10F7, Q57 STD80N10F7, U1 AD7606C-16BSTZ, U2 AP2112K-3.3, U3 USBLC6-2SC6, U30 LMZ14202HTZX/NOPB, U31 LMZ14202HTZX/NOPB, U40 OPA197IDBVR, U41 OPA197IDBVR, U42 TLV3501AIDBVR, U44 TPS60403DBVR, U51 UCC27282DR, U52 UCC27282DR, U53 UCC27282DR, U54 UCC27282DR, U60 OPA197IDBVR, U61 OPA197IDBVR, U62 TLV3501AIDBVR, U70 OPA197IDBVR, U71 OPA197IDBVR, U72 OPA197IDBVR, U73 OPA197IDBVR

Commit message: Remove the redundant 2.2uF/100nF bypass pairs beside both GDT bridges
C527/C528 (GDT 1) and C567/C568 (GDT 2) sat beside the eight-part
22uF 2220 reservoir banks and were fed from the VBAT bus by a back-side
detour (via, B.Cu run, via) per bridge. Eight 2220 MLCCs in parallel are
already within a few millimetres of each bridge and have lower combined
inductance than a single 0805 or 1210, so the small parts were neither
closer nor lower impedance at any frequency. Removed rather than
rerouted.

Circuit contract (docs/circuit.json) drops the four parts; the routing
recipe drops their placements, pads and the 20 detour copper objects,
lists them as removed footprints and carries the new contract hash. The
output-stage schematic block no longer draws the "Local bypass" bank;
schematic, symbol library and PDF regenerated. OUTPUT-STAGE.md and
CERAMIC-RESERVOIRS.md updated (the latter previously said to keep these
parts).

ERC 0, DRC 0/0 with 0 parity issues (kicad-cli and kicadmium), lint
0 open; the eight width-step waivers at the removed feeds resolved and
were pruned (141 -> 133 exceptions). Before/after crops in
docs/gdt-bypass-caps-*.png.

Co-Authored-By: Claude Fable 5.1 <noreply@anthropic.com>
Parts:
- removed C527: 2.2uF 50V X7R, Tesla:C_1210_3225Metric, symbol Tesla:C527
- removed C528: 100nF 50V, Tesla:C_0805_2012Metric, symbol Tesla:C528
- removed C567: 2.2uF 50V X7R, Tesla:C_1210_3225Metric, symbol Tesla:C567
- removed C568: 100nF 50V, Tesla:C_0805_2012Metric, symbol Tesla:C568
Other:
- note removed: "Local bypass"

Commit message: Remove C333, the lone 22uF 1812 beside the battery reservoir
C333 hung on its own 2.5 mm dead-end stub off the VBAT bus, next to the
eight-part 22uF 2220 battery reservoir (C335-C342) on the same rail. It
added about 12 percent to a 176uF nominal bank and nothing else, a
leftover from the removed 24 V converter. Removed from the circuit
contract, recipe (placement, pads, two stub tracks, removed-footprints
list, contract hash), placement files and the schematic generator's
"Local rail bypass" bank; schematic, symbol library and PDF regenerated;
POWER-DESIGN.md updated.

ERC 0, DRC 0/0 with 0 parity issues (kicad-cli and kicadmium), lint
0 open; the two width-step waivers at the stub resolved and were pruned
(133 -> 131 exceptions). Before/after crops in docs/c333-*.png.

Co-Authored-By: Claude Fable 5.1 <noreply@anthropic.com>
Parts:
- removed C333: 22uF 50V, Tesla:C_1812_4532Metric, symbol Tesla:C333
Other:
- note removed: "Local rail bypass"
- moved on the sheet: C1, C10, C11, C12, C13, C14, C15, C16, C17, C18, C2, C22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
